File: eagle/caracas/untitled.brd (EAGLE design)
At the start: 84.8 x 43.2 mm, 8 parts, among them IC1 4027N

Commit message: Save the board again.
Parts:
- added R2, R4: 10k, rcl:0207/10
- added R3: 86, rcl:0207/10
- added T1: 2N2222, transistor:TO18
Connections:
- new net +12V: T1.3
- new net N$1: IC1.7
- new net N$2: R3.1, T1.2
- new net N$4: IC1.4, R4.2, T1.1
- net +12V_IGN: now also R2.2; no longer IC1.7
- net GND: now also R2.1, R4.1
- net RPI-OFFSIGNAL: now also R3.2; no longer IC1.4
Routing:
- net RPI-OFFSIGNAL: track 23.7 -> 16.5 mm
- net +12V_IGN: track 94.1 -> 88.7 mm
Changed lines of the file:
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@@
 <element name="U$2" library="caracas" package="CD2109" value="CD2109" x="48.26" y="7.62" rot="R180"/>
 <element name="U$3" library="caracas" package="MKDS3" value="MKDS3" x="12.7" y="7.62"/>
+<element name="R2" library="rcl" package="0207/10" value="10k" x="6.35" y="-3.81"/>
+<element name="R3" library="rcl" package="0207/10" value="86" x="6.35" y="-8.89"/>
+<element name="R4" library="rcl" package="0207/10" value="10k" x="6.35" y="-13.97"/>
+<element name="T1" library="transistor" package="TO18" value="2N2222" x="5.08" y="-24.13"/>
 </elements>
 <signals>
@@
 <wire x1="16.51" y1="7.62" x2="15.26" y2="7.64" width="0.508" layer="16"/>
 <wire x1="36.83" y1="10.16" x2="36.695" y2="10.52" width="0.508" layer="16"/>
+<contactref element="R2" pad="1"/>
+<contactref element="R4" pad="1"/>
+<wire x1="1.27" y1="-3.81" x2="15.26" y2="7.64" width="0" layer="19" extent="1-1"/>
+<wire x1="1.27" y1="-13.97" x2="1.27" y2="-3.81" width="0" layer="19" extent="1-1"/>
 </signal>
 <signal name="RPI-OFFSIGNAL">
 <contactref element="CON1" pad="18"/>
-<contactref element="IC1" pad="4"/>
-<wire x1="60.96" y1="26.67" x2="55.88" y2="31.75" width="0.508" layer="16"/>
 <wire x1="77.47" y1="26.67" x2="60.96" y2="26.67" width="0.508" layer="16"/>
+<contactref element="R3" pad="2"/>
+<wire x1="11.43" y1="-8.89" x2="60.96" y2="26.67" width="0" layer="19" extent="16-16"/>
 </signal>
 <signal name="VCC">
@@
 <signal name="+12V_IGN">
 <contactref element="U$3" pad="P$2"/>
-<contactref element="IC1" pad="7"/>
-<wire x1="67.31" y1="27.94" x2="63.5" y2="31.75" width="0.508" layer="16"/>
 <wire x1="78.74" y1="27.94" x2="67.31" y2="27.94" width="0.508" layer="16"/>
 <wire x1="78.74" y1="10.16" x2="78.74" y2="27.94" width="0.508" layer="16"/>
@@
 <wire x1="21.59" y1="7.62" x2="69.85" y2="7.62" width="0.508" layer="16"/>
 <wire x1="21.59" y1="7.62" x2="20.34" y2="7.64" width="0.508" layer="16"/>
+<contactref element="R2" pad="2"/>
+<wire x1="11.43" y1="-3.81" x2="20.34" y2="7.64" width="0" layer="19" extent="1-1"/>
 </signal>
 <signal name="+5V">
@@
 <wire x1="43.18" y1="10.16" x2="43.045" y2="10.52" width="0.508" layer="16"/>
 </signal>
+<signal name="N$4">
+<contactref element="IC1" pad="4"/>
+<contactref element="T1" pad="1"/>
+<contactref element="R4" pad="2"/>
+<wire x1="11.43" y1="-13.97" x2="55.88" y2="31.75" width="0" layer="19" extent="1-1"/>
+<wire x1="3.81" y1="-25.4" x2="11.43" y2="-13.97" width="0" layer="19" extent="1-1"/>
+</signal>
+<signal name="N$1">
+<contactref element="IC1" pad="7"/>
+</signal>
+<signal name="N$2">
+<contactref element="R3" pad="1"/>
+<contactref element="T1" pad="2"/>
+<wire x1="1.27" y1="-8.89" x2="6.35" y2="-25.4" width="0" layer="19" extent="1-1"/>
+</signal>
+<signal name="+12V">
+<contactref element="T1" pad="3"/>
+</signal>
 </signals>

Commit message: WIP on electronics schematics.
Parts:
- removed C1: 220µ, rcl:C025-024X044
- removed C2: 10µ, rcl:C025-024X044
- removed R2: 10k, rcl:0207/10
- removed U$1: NCS12S1205C, caracas:NCS12S1205C
- added R5, R6, R7, R8: (no value), rcl:0309/12
Connections:
- removed net N$1: IC1.7
- new net +3.3V: IC1.16, R5.1, R6.2
- new net +3.3V1: IC1.7, R7.1, R8.2
- net +12V_IGN: now also R7.2; no longer R2.2
- net +5V: now also R5.2; no longer C1.1, U$1.+VOUT
- net GND: now also R6.1, R8.1; no longer C1.2, C2.1, R2.1, U$1.-VIN1, U$1.-VIN2, U$1.0V
- net N$4: no longer IC1.4
- net POWER_STATE: no longer U$1.CONTROL
- net VCC: no longer C2.2, IC1.16, U$1.+VIN1, U$1.+VIN2
Routing:
- net VCC: track 85.4 -> 32.4 mm
- net GND: track 170.1 -> 125.5 mm
- net +5V: track 211.4 -> 167.9 mm
- net POWER_STATE: track 59.5 -> 36.2 mm
Changed lines of the file:
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@@
 <attribute name="OC_FARNELL" value="unknown" x="123.19" y="54.61" size="1.778" layer="27" rot="R90" display="off"/>
 </element>
-<element name="U$1" library="caracas" package="NCS12S1205C" value="NCS12S1205C" x="17.78" y="30.48"/>
-<element name="C1" library="rcl" package="C025-024X044" value="220µ" x="20.32" y="16.51" rot="R90"/>
-<element name="C2" library="rcl" package="C025-024X044" value="10µ" x="15.24" y="16.51" rot="R90"/>
 <element name="IC1" library="40xx" package="DIL16" value="4027N" x="57.15" y="35.56"/>
 <element name="U$2" library="caracas" package="CD2109" value="CD2109" x="48.26" y="7.62" rot="R180"/>
 <element name="U$3" library="caracas" package="MKDS3" value="MKDS3" x="12.7" y="7.62"/>
-<element name="R2" library="rcl" package="0207/10" value="10k" x="6.35" y="-3.81"/>
 <element name="R3" library="rcl" package="0207/10" value="86" x="6.35" y="-8.89"/>
 <element name="R4" library="rcl" package="0207/10" value="10k" x="6.35" y="-13.97"/>
 <element name="T1" library="transistor" package="TO18" value="2N2222" x="5.08" y="-24.13"/>
+<element name="R5" library="rcl" package="0309/12" value="" x="7.62" y="-31.75"/>
+<element name="R6" library="rcl" package="0309/12" value="" x="7.62" y="-38.1"/>
+<element name="R7" library="rcl" package="0309/12" value="" x="7.62" y="-44.45"/>
+<element name="R8" library="rcl" package="0309/12" value="" x="7.62" y="-50.8"/>
 </elements>
 <signals>
 <signal name="GND">
-<contactref element="C2" pad="1"/>
-<contactref element="U$1" pad="0V"/>
-<contactref element="C1" pad="2"/>
-<contactref element="U$1" pad="-VIN1"/>
-<contactref element="U$1" pad="-VIN2"/>
 <contactref element="CON1" pad="6"/>
 <contactref element="U$2" pad="P4"/>
@@
 <contactref element="IC1" pad="6"/>
 <wire x1="15.24" y1="8.89" x2="15.24" y2="12.7" width="0.508" layer="16"/>
-<wire x1="15.24" y1="12.7" x2="15.24" y2="15.24" width="0.508" layer="16"/>
 <wire x1="15.24" y1="8.89" x2="15.26" y2="7.64" width="0.508" layer="16"/>
-<wire x1="15.24" y1="12.7" x2="20.32" y2="17.78" width="0.508" layer="16"/>
-<wire x1="10.16" y1="22.86" x2="7.62" y2="22.86" width="0.508" layer="16"/>
-<wire x1="10.16" y1="22.86" x2="12.7" y2="25.4" width="0.508" layer="16"/>
-<wire x1="12.7" y1="25.4" x2="25.4" y2="38.1" width="0.508" layer="16"/>
-<wire x1="12.7" y1="25.4" x2="20.32" y2="17.78" width="0.508" layer="16"/>
 <wire x1="55.88" y1="34.29" x2="53.34" y2="31.75" width="0.508" layer="16"/>
 <wire x1="58.42" y1="31.75" x2="55.88" y2="34.29" width="0.508" layer="16"/>
@@
 <wire x1="16.51" y1="7.62" x2="15.26" y2="7.64" width="0.508" layer="16"/>
 <wire x1="36.83" y1="10.16" x2="36.695" y2="10.52" width="0.508" layer="16"/>
-<contactref element="R2" pad="1"/>
 <contactref element="R4" pad="1"/>
-<wire x1="1.27" y1="-3.81" x2="15.26" y2="7.64" width="0" layer="19" extent="1-1"/>
-<wire x1="1.27" y1="-13.97" x2="1.27" y2="-3.81" width="0" layer="19" extent="1-1"/>
+<contactref element="R6" pad="1"/>
+<contactref element="R8" pad="1"/>
+<wire x1="1.27" y1="-38.1" x2="1.27" y2="-50.8" width="0" layer="19" extent="1-1"/>
+<wire x1="1.27" y1="-13.97" x2="1.27" y2="-38.1" width="0" layer="19" extent="1-1"/>
+<wire x1="15.26" y1="7.64" x2="1.27" y2="-13.97" width="0" layer="19" extent="1-1"/>
 </signal>
 <signal name="RPI-OFFSIGNAL">
@@
 </signal>
 <signal name="VCC">
-<contactref element="C2" pad="2"/>
-<contactref element="U$1" pad="+VIN1"/>
-<contactref element="U$1" pad="+VIN2"/>
-<contactref element="IC1" pad="16"/>
 <contactref element="U$3" pad="P$1"/>
 <wire x1="5.1" y1="7.64" x2="11.43" y2="13.97" width="0.508" layer="16"/>
-<wire x1="11.43" y1="13.97" x2="15.24" y2="17.78" width="0.508" layer="16"/>
-<wire x1="41.91" y1="39.37" x2="48.26" y2="39.37" width="0.508" layer="16"/>
-<wire x1="40.64" y1="40.64" x2="41.91" y2="39.37" width="0.508" layer="16"/>
-<wire x1="12.7" y1="40.64" x2="40.64" y2="40.64" width="0.508" layer="16"/>
-<wire x1="10.16" y1="38.1" x2="12.7" y2="40.64" width="0.508" layer="16"/>
-<wire x1="10.16" y1="38.1" x2="7.62" y2="38.1" width="0.508" layer="16"/>
 <wire x1="3.81" y1="21.59" x2="11.43" y2="13.97" width="0.508" layer="16"/>
 <wire x1="3.81" y1="34.29" x2="3.81" y2="21.59" width="0.508" layer="16"/>
-<wire x1="7.62" y1="38.1" x2="3.81" y2="34.29" width="0.508" layer="16"/>
 </signal>
 <signal name="POWER_STATE">
 <contactref element="IC1" pad="1"/>
-<contactref element="U$1" pad="CONTROL"/>
 <contactref element="R1" pad="1"/>
 <wire x1="48.26" y1="31.75" x2="48.26" y2="25.4" width="0.508" layer="16"/>
-<wire x1="21.59" y1="39.37" x2="5.08" y2="22.86" width="0.508" layer="16"/>
 <wire x1="40.64" y1="39.37" x2="21.59" y2="39.37" width="0.508" layer="16"/>
 <wire x1="48.26" y1="31.75" x2="40.64" y2="39.37" width="0.508" layer="16"/>
@@
 <wire x1="21.59" y1="7.62" x2="69.85" y2="7.62" width="0.508" layer="16"/>
 <wire x1="21.59" y1="7.62" x2="20.34" y2="7.64" width="0.508" layer="16"/>
-<contactref element="R2" pad="2"/>
-<wire x1="11.43" y1="-3.81" x2="20.34" y2="7.64" width="0" layer="19" extent="1-1"/>
+<contactref element="R7" pad="2"/>
+<wire x1="20.34" y1="7.64" x2="13.97" y2="-44.45" width="0" layer="19" extent="1-1"/>
 </signal>
 <signal name="+5V">
 <contactref element="U$3" pad="P$3"/>
-<contactref element="C1" pad="1"/>
-<contactref element="U$1" pad="+VOUT"/>
 <contactref element="CON1" pad="2"/>
 <contactref element="CON1" pad="4"/>
@@
 <wire x1="40.64" y1="10.16" x2="40.505" y2="10.52" width="0.508" layer="16"/>
 <wire x1="41.91" y1="10.16" x2="43.18" y2="10.16" width="0.508" layer="16"/>
-<wire x1="36.83" y1="15.24" x2="20.32" y2="15.24" width="0.508" layer="16"/>
 <wire x1="41.91" y1="10.16" x2="36.83" y2="15.24" width="0.508" layer="16"/>
 <wire x1="41.91" y1="10.16" x2="41.775" y2="10.52" width="0.508" layer="16"/>
-<wire x1="30.48" y1="25.4" x2="30.48" y2="38.1" width="0.508" layer="16"/>
-<wire x1="20.32" y1="15.24" x2="30.48" y2="25.4" width="0.508" layer="16"/>
 <wire x1="77.47" y1="8.89" x2="77.47" y2="7.62" width="0.508" layer="16"/>
 <wire x1="77.47" y1="7.62" x2="77.47" y2="6.35" width="0.508" layer="16"/>
@@
 <wire x1="77.47" y1="7.62" x2="81.28" y2="7.62" width="0.508" layer="16"/>
 <wire x1="43.18" y1="10.16" x2="43.045" y2="10.52" width="0.508" layer="16"/>
+<contactref element="R5" pad="2"/>
+<wire x1="13.97" y1="-31.75" x2="13.97" y2="5.08" width="0" layer="19" extent="16-16"/>
 </signal>
 <signal name="N$4">
-<contactref element="IC1" pad="4"/>
 <contactref element="T1" pad="1"/>
 <contactref element="R4" pad="2"/>
-<wire x1="11.43" y1="-13.97" x2="55.88" y2="31.75" width="0" layer="19" extent="1-1"/>
-<wire x1="3.81" y1="-25.4" x2="11.43" y2="-13.97" width="0" layer="19" extent="1-1"/>
-</signal>
-<signal name="N$1">
-<contactref element="IC1" pad="7"/>
+<wire x1="11.43" y1="-13.97" x2="3.81" y2="-25.4" width="0" layer="19" extent="1-1"/>
 </signal>
 <signal name="N$2">
@@
 <contactref element="T1" pad="3"/>
 </signal>
+<signal name="+3.3V">
+<contactref element="IC1" pad="16"/>
+<contactref element="R5" pad="1"/>
+<contactref element="R6" pad="2"/>
+<wire x1="13.97" y1="-38.1" x2="48.26" y2="39.37" width="0" layer="19" extent="1-1"/>
+<wire x1="1.27" y1="-31.75" x2="13.97" y2="-38.1" width="0" layer="19" extent="1-1"/>
+</signal>
+<signal name="+3.3V1">
+<contactref element="R7" pad="1"/>
+<contactref element="R8" pad="2"/>
+<contactref element="IC1" pad="7"/>
+<wire x1="13.97" y1="-50.8" x2="63.5" y2="31.75" width="0" layer="19" extent="1-1"/>
+<wire x1="1.27" y1="-44.45" x2="13.97" y2="-50.8" width="0" layer="19" extent="1-1"/>
+</signal>
 </signals>

Commit message: More WIP on the electronics schematics, closing in...
Parts:
- removed T1: 2N2222, transistor:TO18
- removed U$3: MKDS3, caracas:MKDS3
- added Q1: IRFP250, transistor-power:TO-247AD-V
- added R10, R11, R12, R13, R14, R15, R2, R9: (no value), rcl:0207/10
- added U$1: MCP3008-I/P, mpc3008:DIP254P762X432-16
- added X1, X2, X5, X6: 22-23-2021, con-molex:22-23-2021
- added X3, X4: 22-23-2041, con-molex:22-23-2041
- R1, R4: value 10k -> (none)
- R3: value 86 -> (none)
- R5, R6, R7, R8: device rcl:0309/12 -> rcl:0207/10
- U$2: value CD2109 -> MKDS3; device caracas:CD2109 -> caracas:MKDS3
- moved R4 88.0 mm to (88.9, 16.5)
- moved R7 86.9 mm to (47.0, 33.0), turned to 270 degrees
- moved R5 85.3 mm to (76.2, 19.1)
- moved R6 83.9 mm to (52.1, 33.0), turned to 270 degrees
- moved R8 71.4 mm to (14.0, 20.3), turned to 90 degrees
- moved R3 46.8 mm to (41.9, 21.6), turned to 90 degrees
- moved R1 40.7 mm to (88.9, 19.1), turned to 180 degrees
- moved U$2 34.3 mm to (82.5, 8.89)
- moved CON1 30.7 mm to (50.8, 8.89), turned to 180 degrees
- moved IC1 15.5 mm to (54.6, 20.3)
Connections:
- removed net +12V: T1.3
- removed net RPI-OFFSIGNAL: CON1.18, R3.2
- new net +5V_SW_GND: CON1.6, Q1.D
- new net ANA_0: R8.1, U$1.1, X4.3
- new net ANA_1: R9.1, U$1.2, X4.2
- new net N$1: Q1.G, R3.2
- new net N$10: CON1.12, R13.1, X3.2
- new net N$11: IC1.14, R11.2
- new net N$12: IC1.10, IC1.11, IC1.12, IC1.13, IC1.9, R10.2
- new net N$13: IC1.15, R12.2
- new net N$5: CON1.19, U$1.11
- new net N$6: CON1.24, U$1.10
- new net N$7: CON1.8, R15.1, X3.4
- new net N$8: CON1.10, R14.1, X3.3
- new net N$9: IC1.3, IC1.5, IC1.6, R6.2
- new net SUICIDE: CON1.11, IC1.4
- net +12V_IGN: now also R2.1, U$2.P$3; no longer R7.2, U$3.P$2
- net +3.3V: now also R1.2, R4.1, R8.2, R9.2, U$1.15, U$1.16, X3.1, X4.4; no longer R5.1, R6.2
- net +3.3V1: now also R2.2, R5.1; no longer R7.1, R8.2
- net +5V: now also R1.1, X1.1, X1.2; no longer R5.2, U$2.P7, U$2.P8, U$2.P9, U$3.P$3
- net GND: now also Q1.S, R10.1, R11.1, R12.1, R13.2, R14.2, R15.2, R4.2, R5.2, R7.1, U$1.14, U$1.9, U$2.P$1, X4.1, X5.1, X5.2, X6.1, X6.2; no longer CON1.6, IC1.3, IC1.5, IC1.6, R4.1, R8.1, U$2.P10, U$2.P12, U$2.P4, U$2.P5, U$2.P6, U$3.P$4
- net N$2: now also IC1.2, R7.2; no longer R3.1, T1.2
- net N$3: now also CON1.5, U$1.13; no longer CON1.16, R1.2
- net N$4: now also CON1.21, U$1.12; no longer R4.2, T1.1
- net POWER_STATE: now also CON1.16, R3.1; no longer R1.1
- net VCC: now also U$2.P$2, X2.1, X2.2; no longer U$3.P$1
Routing:
- net +5V_SW_GND: track 0.00 -> 126.5 mm
- net +3.3V: track 0.00 -> 126.4 mm
- net GND: track 125.5 -> 0.00 mm
- net +5V: track 167.9 -> 50.7 mm
- net N$7: track 0.00 -> 98.8 mm
- net +12V_IGN: track 88.7 -> 9.68 mm
- net N$3: track 32.9 -> 106.5 mm
- net N$8: track 0.00 -> 64.7 mm
- net N$10: track 0.00 -> 61.3 mm
- net N$5: track 0.00 -> 30.0 mm
- net N$4: track 0.00 -> 26.1 mm
- net N$9: track 0.00 -> 22.5 mm
- net POWER_STATE: track 36.2 -> 14.2 mm
- net ANA_1: track 0.00 -> 20.8 mm
- net N$6: track 0.00 -> 18.6 mm
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- added copper zone on layer 16, net GND
Other:
- board size 84.8 x 43.2 mm -> 100 x 49.5 mm

Commit message: Schematic and board finished (at least R1)
Parts:
- Q1: value IRFP250 -> IRLZ44Z; device transistor-power:TO-247AD-V -> transistor-power:TO220BH
- moved R8 86.4 mm to (100.3, 20.3), turned to 270 degrees
- moved R9 81.3 mm to (97.8, 20.3), turned to 270 degrees
- moved X4 75.7 mm to (82.5, 38.1)
- moved X3 73.4 mm to (92.7, 38.1), turned to 180 degrees
- moved X1 66.1 mm to (27.9, 25.4)
- moved X5 66.1 mm to (27.9, 40.6)
- moved R13 65.1 mm to (67.3, 43.2), turned to 180 degrees
- moved U$2 63.5 mm to (19.1, 10.2), turned to 0 degrees
- moved X2 62.2 mm to (7.62, 25.4)
- moved X6 62.2 mm to (7.62, 40.6)
- moved R14 61.9 mm to (67.3, 40.6), turned to 180 degrees
- moved R15 58.6 mm to (67.3, 38.1), turned to 180 degrees
- moved R4 43.2 mm to (49.5, 34.3), turned to 180 degrees
- moved R2 42.2 mm to (34.3, 11.4), turned to 90 degrees
- moved R1 41.4 mm to (49.5, 31.8), turned to 0 degrees
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Connections:
- net +12V_IGN: now also U$2.P$4; no longer U$2.P$3
- net +3.3V: now also X4.1, X4.2; no longer X3.1, X4.4
- net ANA_1: now also X4.4; no longer X4.2
- net GND: no longer X4.1
- net VCC: now also U$2.P$3; no longer U$2.P$2
Routing:
- net +5V_SW_GND: track 126.5 -> 22.0 mm
- net SUICIDE: track 6.35 -> 75.8 mm
- net POWER_STATE: track 14.2 -> 73.1 mm
- net N$13: track 4.34 -> 37.0 mm
- net N$7: track 98.8 -> 68.3 mm
- net N$8: track 64.7 -> 36.5 mm
- net ANA_0: track 13.4 -> 39.7 mm
- net N$1: track 12.9 -> 36.4 mm
- net +3.3V: track 126.4 -> 144.9 mm
- net ANA_1: track 20.8 -> 32.5 mm
- net N$6: track 18.6 -> 29.1 mm
- net N$5: track 30.0 -> 20.4 mm
- net +5V: track 50.7 -> 42.5 mm
- net N$12: track 14.5 -> 22.2 mm
- net N$3: track 106.5 -> 98.8 mm
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Other:
- board size 100 x 49.5 mm -> 110.2 x 53.3 mm
